File: kojak/kojak.sch (KiCad schematic (older format))
At the start: 23 parts, among them Q1 BC546, Q2 BC546, Q3 BC557, Q4 TIP31C, SW1 MODE

Commit message: rescue
Parts:
- BT1: symbol Device:Battery -> kojak-rescue:Battery-Device
- C1, C2, C3, C4: symbol Device:CP -> kojak-rescue:CP-Device
- C5, C6: symbol Device:C -> kojak-rescue:C-Device
- D1, D2: symbol Device:LED -> kojak-rescue:LED-Device
- LS1: symbol Device:Speaker -> kojak-rescue:Speaker-Device
- Q1, Q2: symbol Transistor_BJT:BC546 -> kojak-rescue:BC546-Transistor_BJT
- Q3: symbol Transistor_BJT:BC557 -> kojak-rescue:BC557-Transistor_BJT
- Q4: symbol Transistor_BJT:TIP41C -> kojak-rescue:TIP41C-Transistor_BJT
- R1, R2, R3, R4, R5, R6, R7, R8: symbol Device:R -> kojak-rescue:R-Device
- SW1: symbol Switch:SW_SPDT -> kojak-rescue:SW_SPDT-Switch
Changed lines of the file:
@@
 $EndDescr
 $Comp
-L Transistor_BJT:BC546 Q1
+L kojak-rescue:BC546-Transistor_BJT Q1
 U 1 1 5DDDC5A6
 P 3075 2975
@@
 $EndComp
 $Comp
-L Transistor_BJT:BC546 Q2
+L kojak-rescue:BC546-Transistor_BJT Q2
 U 1 1 5DDDCBE1
 P 4500 2975
@@
 $EndComp
 $Comp
-L Device:CP C2
+L kojak-rescue:CP-Device C2
 U 1 1 5DDDE1A8
 P 3275 2650
@@
 $EndComp
 $Comp
-L Device:R R2
+L kojak-rescue:R-Device R2
 U 1 1 5DDDF0A3
 P 3575 2075
@@
 $EndComp
 $Comp
-L Device:R R4
+L kojak-rescue:R-Device R4
 U 1 1 5DDE0F87
 P 4600 2350
@@
 $EndComp
 $Comp
-L Device:R R1
+L kojak-rescue:R-Device R1
 U 1 1 5DDE131E
 P 2975 2350
@@
 $EndComp
 $Comp
-L Device:LED D1
+L kojak-rescue:LED-Device D1
 U 1 1 5DDE197B
 P 2975 1925
@@
 $EndComp
 $Comp
-L Device:LED D2
+L kojak-rescue:LED-Device D2
 U 1 1 5DDE2C4A
 P 4600 1925
@@
 Connection ~ 3575 2650
 $Comp
-L Device:CP C3
+L kojak-rescue:CP-Device C3
 U 1 1 5DDDD48B
 P 4200 2650
@@
 	3025 4575 3025 4800
 $Comp
-L Device:C C5
+L kojak-rescue:C-Device C5
 U 1 1 5DE158B7
 P 4200 5000
@@
 $EndComp
 $Comp
-L Transistor_BJT:BC557 Q3
+L kojak-rescue:BC557-Transistor_BJT Q3
 U 1 1 5DDDA224
 P 3125 5000
@@
 $EndComp
 $Comp
-L Device:C C6
+L kojak-rescue:C-Device C6
 U 1 1 5DE17E38
 P 4450 5225
@@
 	4900 4800 4900 5000
 $Comp
-L Device:CP C4
+L kojak-rescue:CP-Device C4
 U 1 1 5DE29061
 P 5750 2000
@@
 $EndComp
 $Comp
-L Device:R R5
+L kojak-rescue:R-Device R5
 U 1 1 5DE29718
 P 5525 2650
@@
 $EndComp
 $Comp
-L Device:R R6
+L kojak-rescue:R-Device R6
 U 1 1 5DE29C64
 P 3450 4775
@@
 Connection ~ 2975 1700
 $Comp
-L Device:CP C1
+L kojak-rescue:CP-Device C1
 U 1 1 5DE3576B
 P 1650 2775
@@
 	1650 2925 1650 3075
 $Comp
-L Device:R R3
+L kojak-rescue:R-Device R3
 U 1 1 5DE37F7C
 P 3900 2075
@@
 $EndComp
 $Comp
-L Device:R R7
+L kojak-rescue:R-Device R7
 U 1 1 5DE388ED
 P 3825 5000
@@
 $EndComp
 $Comp
-L Device:R R8
+L kojak-rescue:R-Device R8
 U 1 1 5DE394DF
 P 6425 2000
@@
 $EndComp
 $Comp
-L Transistor_BJT:TIP41C Q4
+L kojak-rescue:TIP41C-Transistor_BJT Q4
 U 1 1 5DE19CEE
 P 4800 5450
@@
 $EndComp
 $Comp
-L Device:Battery BT1
+L kojak-rescue:Battery-Device BT1
 U 1 1 5DE79479
 P 1200 2775
@@
 	1200 3075 1650 3075
 $Comp
-L Device:Speaker LS1
+L kojak-rescue:Speaker-Device LS1
 U 1 1 5DE85C66
 P 5100 4700
@@
 	5900 2000 6000 2000
 $Comp
-L power:GND #PWR0101
+L kojak-rescue:GND-power #PWR0101
 U 1 1 5DE9DD96
 P 2975 3300
@@
 $EndComp
 $Comp
-L power:VCC #PWR0102
+L kojak-rescue:VCC-power #PWR0102
 U 1 1 5DE9EFDF
 P 2975 1575
@@
 	2975 3175 2975 3225
 $Comp
-L power:GND #PWR0103
+L kojak-rescue:GND-power #PWR0103
 U 1 1 5DEC0F44
 P 6650 2000
@@
 	4600 3175 4600 3225
 $Comp
-L power:VCC #PWR0104
+L kojak-rescue:VCC-power #PWR0104
 U 1 1 5DEC82DF
 P 5525 2000
@@
 	5675 2650 6100 2650
 $Comp
-L power:VCC #PWR0105
+L kojak-rescue:VCC-power #PWR0105
 U 1 1 5DED7C6F
 P 1650 2350
@@
 	1650 2475 1650 2350
 $Comp
-L power:GND #PWR0106
+L kojak-rescue:GND-power #PWR0106
 U 1 1 5DEDAC94
 P 1650 3150
@@
 	2575 6050 5725 6050
 $Comp
-L power:GND #PWR0107
+L kojak-rescue:GND-power #PWR0107
 U 1 1 5DF03230
 P 4900 5800
@@
 	4900 5650 4900 5800
 $Comp
-L power:VCC #PWR0108
+L kojak-rescue:VCC-power #PWR0108
 U 1 1 5DF0B033
 P 4900 4550
@@
 	4900 4700 4900 4550
 $Comp
-L power:VCC #PWR0109
+L kojak-rescue:VCC-power #PWR0109
 U 1 1 5DF0CC2E
 P 3025 4575
@@
 	6000 2000 6000 2050
 $Comp
-L pspice:0 #GND0101
+L kojak-rescue:0-pspice #GND0101
 U 1 1 5DE7E19A
 P 1175 3900
@@
 $EndComp
 $Comp
-L power:GND #PWR0110
+L kojak-rescue:GND-power #PWR0110
 U 1 1 5DE7E79F
 P 1300 3900
@@
 	1175 3900 1300 3900
 $Comp
-L Switch:SW_SPDT SW1
+L kojak-rescue:SW_SPDT-Switch SW1
 U 1 1 5DE7E706
 P 6100 2250
